File: baremetal/DogFeeder/kicad/PowerBankAlwaysActive/PowerBankAlwaysActive.sch (KiCad schematic (older format))
At the start: 17 parts, among them J1 Conn_01x02_Female, J2 Conn_01x02_Female, Q1 BC817, U1 ICM7555xB

Commit message: update to cctv & test-pcb board
Parts:
- added R6: 0R, Resistor_SMD:R_1206_3216Metric_Pad1.30x1.75mm_HandSolder, symbol Device:R
- added TP1, TP2, TP3, TP4: TestPoint, Connector_PinHeader_2.54mm:PinHeader_1x01_P2.54mm_Vertical, symbol Connector:TestPoint
- C1: footprint Capacitor_Tantalum_SMD:CP_EIA-1608-10_AVX-L_Pad1.25x1.05mm_HandSolder -> Capacitor_SMD:C_1206_3216Metric
Connections:
- net +5V: now also R6.2, TP2.1; no longer U1.4 (R)
- net GND: now also TP1.1
- net output: now also TP4.1
- net trig: now also TP3.1
- net disch: now reaches D1.2 (A), R1.2, R2.1, U1.7 (DIS)
- new net: R6.1, U1.4 (R)
Changed lines of the file:
@@
-	1    0    0    -1
-$EndComp
-$Comp
-L power:+5V #PWR01
-U 1 1 61BC4BAE
-P 3050 2700
-F 0 "#PWR01" H 3050 2550 50  0001 C CNN
-F 1 "+5V" H 3065 2873 50  0000 C CNN
-F 2 "" H 3050 2700 50  0001 C CNN
-F 3 "" H 3050 2700 50  0001 C CNN
-	1    3050 2700
 	1    0    0    -1
 $EndComp
@@
 Wire Wire Line
 	3800 2900 3800 3200
-Wire Wire Line
-	3300 2700 3050 2700
 $Comp
 L Device:R R2
@@
 F 0 "C1" H 4815 3046 50  0000 L CNN
 F 1 "10uf" H 4815 2955 50  0000 L CNN
-F 2 "Capacitor_Tantalum_SMD:CP_EIA-1608-10_AVX-L_Pad1.25x1.05mm_HandSolder" H 4738 2850 50  0001 C CNN
+F 2 "Capacitor_SMD:C_1206_3216Metric" H 4738 2850 50  0001 C CNN
 F 3 "~" H 4700 3000 50  0001 C CNN
 	1    4700 3000
@@
 	1    0    0    -1
 $EndComp
+$Comp
+L Connector:TestPoint TP3
+U 1 1 61D4E561
+P 4350 4000
+F 0 "TP3" H 4408 4118 50  0000 L CNN
+F 1 "TestPoint" H 4408 4027 50  0000 L CNN
+F 2 "Connector_PinHeader_2.54mm:PinHeader_1x01_P2.54mm_Vertical" H 4550 4000 50  0001 C CNN
+F 3 "~" H 4550 4000 50  0001 C CNN
+	1    4350 4000
+	1    0    0    -1
+$EndComp
+$Comp
+L Connector:TestPoint TP4
+U 1 1 61D4F9DD
+P 4950 4000
+F 0 "TP4" H 5008 4118 50  0000 L CNN
+F 1 "TestPoint" H 5008 4027 50  0000 L CNN
+F 2 "Connector_PinHeader_2.54mm:PinHeader_1x01_P2.54mm_Vertical" H 5150 4000 50  0001 C CNN
+F 3 "~" H 5150 4000 50  0001 C CNN
+	1    4950 4000
+	1    0    0    -1
+$EndComp
+Wire Wire Line
+	4350 4000 4350 4200
+Wire Wire Line
+	4950 4000 4950 4200
+$Comp
+L Connector:TestPoint TP2
+U 1 1 61D550A7
+P 3900 4000
+F 0 "TP2" H 3958 4118 50  0000 L CNN
+F 1 "TestPoint" H 3958 4027 50  0000 L CNN
+F 2 "Connector_PinHeader_2.54mm:PinHeader_1x01_P2.54mm_Vertical" H 4100 4000 50  0001 C CNN
+F 3 "~" H 4100 4000 50  0001 C CNN
+	1    3900 4000
+	1    0    0    -1
+$EndComp
+$Comp
+L Connector:TestPoint TP1
+U 1 1 61D552E7
+P 3350 4000
+F 0 "TP1" H 3408 4118 50  0000 L CNN
+F 1 "TestPoint" H 3408 4027 50  0000 L CNN
+F 2 "Connector_PinHeader_2.54mm:PinHeader_1x01_P2.54mm_Vertical" H 3550 4000 50  0001 C CNN
+F 3 "~" H 3550 4000 50  0001 C CNN
+	1    3350 4000
+	1    0    0    -1
+$EndComp
+$Comp
+L power:GND #PWR05
+U 1 1 61D5650B
+P 3350 4000
+F 0 "#PWR05" H 3350 3750 50  0001 C CNN
+F 1 "GND" H 3355 3827 50  0000 C CNN
+F 2 "" H 3350 4000 50  0001 C CNN
+F 3 "" H 3350 4000 50  0001 C CNN
+	1    3350 4000
+	1    0    0    -1
+$EndComp
+$Comp
+L power:+5V #PWR06
+U 1 1 61D56E51
+P 3900 4000
+F 0 "#PWR06" H 3900 3850 50  0001 C CNN
+F 1 "+5V" H 3915 4173 50  0000 C CNN
+F 2 "" H 3900 4000 50  0001 C CNN
+F 3 "" H 3900 4000 50  0001 C CNN
+	1    3900 4000
+	-1   0    0    1
+$EndComp
+$Comp
+L Device:R R6
+U 1 1 61D587FE
+P 2950 2950
+F 0 "R6" V 2743 2950 50  0000 C CNN
+F 1 "0R" V 2834 2950 50  0000 C CNN
+F 2 "Resistor_SMD:R_1206_3216Metric_Pad1.30x1.75mm_HandSolder" V 2880 2950 50  0001 C CNN
+F 3 "~" H 2950 2950 50  0001 C CNN
+	1    2950 2950
+	0    1    1    0
+$EndComp
+$Comp
+L power:+5V #PWR01
+U 1 1 61D59630
+P 2800 2950
+F 0 "#PWR01" H 2800 2800 50  0001 C CNN
+F 1 "+5V" H 2815 3123 50  0000 C CNN
+F 2 "" H 2800 2950 50  0001 C CNN
+F 3 "" H 2800 2950 50  0001 C CNN
+	1    2800 2950
+	0    -1   -1   0
+$EndComp
+Wire Wire Line
+	3300 2700 3200 2700
+Wire Wire Line
+	3200 2700 3200 2950
+Wire Wire Line
+	3200 2950 3100 2950
+Text Label 4350 4200 1    50   ~ 0
+trig
+Text Label 4950 4200 1    50   ~ 0
+output
+Text Label 4700 2450 0    50   ~ 0
+disch
 $EndSCHEMATC
