File: baremetal/DogFeeder/kicad/PowerBankAlwaysActive/PowerBankAlwaysActive.kicad_pcb (KiCad board)
At the start: 4 copper layers, 36.8 x 23.4 mm, 17 parts, among them J1 Conn_01x02_Female, J2 Conn_01x02_Female, Q1 BC817, U1 ICM7555xB

Commit message: update to cctv & test-pcb board
Parts:
- added +5: TestPoint, Connector_PinHeader_2.54mm:PinHeader_1x01_P2.54mm_Vertical, F.Cu at (40.9, 42.2)
- added R6: 0R, Resistor_SMD:R_1206_3216Metric_Pad1.30x1.75mm_HandSolder, F.Cu at (42.9, 30.3)
- added gnd: TestPoint, Connector_PinHeader_2.54mm:PinHeader_1x01_P2.54mm_Vertical, F.Cu at (44.9, 42.2)
- added out: TestPoint, Connector_PinHeader_2.54mm:PinHeader_1x01_P2.54mm_Vertical, F.Cu at (37.8, 29.5)
- added trig: TestPoint, Connector_PinHeader_2.54mm:PinHeader_1x01_P2.54mm_Vertical, F.Cu at (33.8, 29.5)
- C1: footprint Capacitor_Tantalum_SMD:CP_EIA-1608-10_AVX-L_Pad1.25x1.05mm_HandSolder -> Capacitor_SMD:C_1206_3216Metric
- moved C2 5.56 mm to (44.7, 27.2), turned to 0 degrees
- moved R5 2.02 mm to (44.7, 24.7)
- moved D2 2.00 mm to (50.5, 24.7)
- moved R4 0.99 mm to (50.0, 30.7)
Connections:
- net Net-(D1-Pad2) renamed /disch
- U1 pad 4: +5V -> Net-(R6-Pad1)
Routing:
- net +5V: track 26.2 -> 17.6 mm
- net /output: track 2.89 -> 10.1 mm
- net Net-(R6-Pad1): track 0.00 -> 4.48 mm
- net /trig: track 20.5 -> 24.3 mm
- net /disch: track 24.9 -> 26.9 mm
- net Net-(D2-Pad1): track 15.8 -> 16.9 mm
- net GND: track 14.0 -> 14.7 mm
Other:
- board text added: "Version 1.1 Gliese"
- board text removed: "Version 1.0 Gliese"

Commit message: finalized powerbank-actiavtor
Other:
- net class Default removed
