File: baremetal/WindowViewer_Battery/kicad/ESP32_BAT/ESP32_BAT.kicad_pcb (KiCad board)
At the start: 2 copper layers, 49 parts, among them J1 Conn_01x04_Male, J2 Conn_01x02_Male, J3 Conn_01x03_Male, Q1 BC817, U1 ESP32-S2-WROVER, U2 AP7365, U3 am2320

Commit message: watersensor 0.1
Parts:
- added H1: MountingHole, MountingHole:MountingHole_2.2mm_M2_DIN965, F.Cu at (86.6, 119.6)
- added H2: MountingHole, MountingHole:MountingHole_2.2mm_M2_DIN965, F.Cu at (68.6, 119.6)
- added H3: MountingHole, MountingHole:MountingHole_2.2mm_M2_DIN965, F.Cu at (77.6, 82.6)
- added J4: Conn_01x02_Male, Connector_PinHeader_2.54mm:PinHeader_1x02_P2.54mm_Vertical, F.Cu at (60.0, 61.4)
- R13: value 0 -> 10k
- TP10, TP11, TP8, TP9: footprint Connector_PinHeader_2.54mm:PinHeader_1x01_P2.54mm_Vertical -> TestPoint:TestPoint_Pad_2.5x2.5mm
- U1: value ESP32-S2-WROVER -> ESP32-WROOM-32; footprint RF_Module:ESP32-S2-WROVER -> RF_Module:ESP32-WROOM-32
- moved C9 120.5 mm to (79.5, 117.6), turned to 90 degrees
- moved C10 117.7 mm to (77.1, 117.6), turned to 90 degrees
- moved Q1 111.3 mm to (70.0, 87.8), turned to -90 degrees
- moved R5 103.7 mm to (77.7, 93.3)
- moved R12 103.7 mm to (71.4, 95.7)
- moved R2 103.7 mm to (69.6, 93.3)
- moved R11 102.8 mm to (70.9, 83.0), turned to 90 degrees
- moved U3 102.2 mm to (69.2, 104.7)
- moved R13 89.1 mm to (65.0, 61.5)
- moved TP12 86.5 mm to (80.7, 88.0)
- moved TP13 83.3 mm to (86.3, 80.5)
- moved TP2 83.3 mm to (86.3, 84.1)
- moved TP3 83.3 mm to (86.3, 87.7)
- moved R14 78.0 mm to (81.4, 95.8), turned to -90 degrees
- moved C2 77.7 mm to (47.9, 42.1), turned to -90 degrees
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Connections:
- R13 pad 1: /sensor/sensor_gnd -> /ESP32_SOLO/IO0
- R13 pad 2: GND -> +3V3
- U1 pad 12: unconnected-(U1-Pad12) -> SENSOR_ON
- U1 pad 13: unconnected-(U1-Pad13) -> CLK
- U1 pad 14: SENSOR_ON -> unconnected-(U1-Pad14)
- U1 pad 15: unconnected-(U1-Pad15) -> GND
- U1 pad 16: unconnected-(U1-Pad16) -> SDA
- U1 pad 17: CLK -> unconnected-(U1-Pad17)
- U1 pad 18: SDA -> unconnected-(U1-Pad18)
- U1 pad 25: unconnected-(U1-Pad25) -> /ESP32_SOLO/IO0
- U1 pad 26: GND -> unconnected-(U1-Pad26)
- U1 pad 27: Net-(C4-Pad1) -> unconnected-(U1-Pad27)
- U1 pad 28: ADC_SNS_IN -> unconnected-(U1-Pad28)
- U1 pad 3: unconnected-(U1-Pad3) -> /ESP32_SOLO/ENABLE
- U1 pad 34: unconnected-(U1-Pad34) -> /ESP32_SOLO/RXD0
- U1 pad 35: unconnected-(U1-Pad35) -> /ESP32_SOLO/TXD0
- U1 pad 37: /ESP32_SOLO/TXD0 -> unconnected-(U1-Pad37)
- U1 pad 38: /ESP32_SOLO/RXD0 -> GND
- U1 pad 39: unconnected-(U1-Pad39) -> GND
- U1 pad 6: unconnected-(U1-Pad6) -> Net-(C4-Pad1)
- U1 pad 9: unconnected-(U1-Pad9) -> ADC_SNS_IN
Routing:
- net CLK: track 0.00 -> 108.2 mm, vias 0 -> 2
- net +5V: track 0.00 -> 101.9 mm, vias 0 -> 1
- net ADC_SNS_IN: track 0.00 -> 94.8 mm, vias 0 -> 4
- net SDA: track 0.00 -> 74.3 mm, vias 0 -> 2
- net GND: track 0.00 -> 61.0 mm, vias 0 -> 29
- net Net-(C4-Pad1): track 6.60 -> 65.3 mm, vias 0 -> 3
- net SENSOR_ON: track 0.00 -> 49.5 mm, vias 0 -> 2
- net /ESP32_SOLO/RXD0: track 14.5 -> 58.3 mm, vias 0 -> 2
- net +3V3: track 2.75 -> 43.4 mm, vias 0 -> 11
- net +BATT: track 10.2 -> 49.3 mm, vias 0 -> 1
- net /ESP32_SOLO/TXD0: track 15.0 -> 49.9 mm, vias 0 -> 1
- net /sensor/sensor_gnd: track 0.00 -> 32.0 mm, vias 0 -> 4
- net /ESP32_SOLO/ENABLE: track 22.8 -> 49.9 mm, vias 0 -> 2
- net /ESP32_SOLO/IO0: track 0.00 -> 15.4 mm
- net Net-(J3-Pad2): track 0.00 -> 8.04 mm
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- added copper zone on In2.Cu, net +3V3
- added copper zone on In1.Cu, net /sensor/sensor_gnd
- added copper zone on B.Cu, net GND
Other:
- board outline added: 50 x 95 mm
- copper layers 2 -> 4
- board text added: "5V"
- board text added: "ADC"
- board text added: "BAT"
- board text added: "Battery Sensor V1.0 2022 Gliese"
- board text added: "IO0"
- board text added: "S_ON"
