File: baremetal/WindowViewer_Battery/kicad/ESP32_BAT/ESP32_SOLO.kicad_sch (KiCad schematic)
At the start: 13 parts

Commit message: battery pcb update, schematic done
Parts:
- removed C?: 1U, Capacitor_SMD:C_1206_3216Metric_Pad1.33x1.80mm_HandSolder, symbol Device:C
- added C1: 1U, Capacitor_SMD:C_1206_3216Metric_Pad1.33x1.80mm_HandSolder, symbol Device:C
- added R2, R5: 4.7k, Resistor_SMD:R_1206_3216Metric_Pad1.30x1.75mm_HandSolder, symbol Device:R
- added TP1, TP12, TP13, TP2, TP3, TP4, TP5, TP6, TP7: TestPoint, Connector_PinHeader_2.54mm:PinHeader_1x01_P2.54mm_Vertical, symbol Connector:TestPoint
- gave numbers to parts that had none: 12
Connections:
- net +3V3: now also R2.2, R5.2
- net ENABLE: now also C1.2, TP4.1
- net GND: now also C1.1, TP13.1
- net RXD0: now also TP6.1
- net TXD0: now also TP7.1
- net at C4.1, R8.1, U1.27 (IO33): now also TP5.1
- net SENSOR_ON: now reaches U1.14 (IO11)
- net SENSOR_ON: now also TP1.1
- net CLK: now reaches U1.17 (IO14)
- net CLK: now also R5.1, TP2.1
- net SDA: now reaches U1.18 (IO15)
- net SDA: now also R2.1, TP3.1
- net ADC_SNS_IN: now reaches U1.28 (IO34)
- net ADC_SNS_IN: now also TP12.1

Commit message: watersensor 0.1
Parts:
- removed U1: ESP32-S2-WROVER, RF_Module:ESP32-S2-WROVER, symbol RF_Module:ESP32-S2-WROVER
- added J4: Conn_01x02_Male, Connector_PinHeader_2.54mm:PinHeader_1x02_P2.54mm_Vertical, symbol Connector:Conn_01x02_Male
- added R13: 10k, Resistor_SMD:R_1206_3216Metric_Pad1.30x1.75mm_HandSolder, symbol Device:R
- added U1: ESP32-WROOM-32, RF_Module:ESP32-WROOM-32, symbol RF_Module:ESP32-WROOM-32
Connections:
- net +3V3: now also R13.2, U1.2 (VDD)
- net ADC_SNS_IN: now also U1.9 (IO33)
- net CLK: now also U1.13 (IO14)
- net ENABLE: now also U1.3 (EN)
- net GND: now also J4.2 (Pin_2), U1.1 (GND), U1.15 (GND), U1.38 (GND), U1.39 (GND)
- net RXD0: now also U1.34 (RXD0/IO3)
- net SDA: now also U1.16 (IO13)
- net SENSOR_ON: now also U1.12 (IO27)
- net TXD0: now also U1.35 (TXD0/IO1)
- net at C4.1, R8.1, TP5.1: now also U1.6 (IO34)
- new net IO0: J4.1 (Pin_1), R13.1, U1.25 (IO0)
- no-connect marks 0 -> 24
Other:
- moved on the sheet: C1, C2, C3, C4, R2, R5, R7, R8, TP1, TP12, TP2, TP3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
