File: baremetal/WindowViewer_Battery/kicad/ESP32_BAT/PSU.kicad_sch (KiCad schematic)
At the start: 10 parts

Commit message: battery pcb update, schematic done
Parts:
- removed C? (x2): 1U, Capacitor_SMD:C_1206_3216Metric_Pad1.33x1.80mm_HandSolder, symbol Device:C
- added C5: 200nf, Capacitor_SMD:C_1206_3216Metric_Pad1.33x1.80mm_HandSolder, symbol Device:C
- added C6: 22pf, Capacitor_SMD:C_1206_3216Metric_Pad1.33x1.80mm_HandSolder, symbol Device:C
- added TP10, TP11, TP8, TP9: TestPoint, Connector_PinHeader_2.54mm:PinHeader_1x01_P2.54mm_Vertical, symbol Connector:TestPoint
- gave numbers to parts that had none: 8
Connections:
- net +3V3: now also TP10.1
- net +5V: now also TP9.1
- net +BATT: now also C5.1, C6.1, TP8.1
- net GND: now also C5.2, C6.2, TP11.1

Commit message: watersensor 0.1
Parts:
- TP10, TP11, TP8, TP9: footprint Connector_PinHeader_2.54mm:PinHeader_1x01_P2.54mm_Vertical -> TestPoint:TestPoint_Pad_2.5x2.5mm
Changed lines of the file:
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@@
       (effects (font (size 1.27 1.27)) (justify left))
     )
-    (property "Footprint" "Connector_PinHeader_2.54mm:PinHeader_1x01_P2.54mm_Vertical" (id 2) (at 123.19 39.37 0)
+    (property "Footprint" "TestPoint:TestPoint_Pad_2.5x2.5mm" (id 2) (at 123.19 39.37 0)
       (effects (font (size 1.27 1.27)) hide)
     )
@@
       (effects (font (size 1.27 1.27)) (justify left))
     )
-    (property "Footprint" "Connector_PinHeader_2.54mm:PinHeader_1x01_P2.54mm_Vertical" (id 2) (at 80.01 39.37 0)
+    (property "Footprint" "TestPoint:TestPoint_Pad_2.5x2.5mm" (id 2) (at 80.01 39.37 0)
       (effects (font (size 1.27 1.27)) hide)
     )
@@
       (effects (font (size 1.27 1.27)) (justify left))
     )
-    (property "Footprint" "Connector_PinHeader_2.54mm:PinHeader_1x01_P2.54mm_Vertical" (id 2) (at 107.95 39.37 0)
+    (property "Footprint" "TestPoint:TestPoint_Pad_2.5x2.5mm" (id 2) (at 107.95 39.37 0)
       (effects (font (size 1.27 1.27)) hide)
     )
@@
       (effects (font (size 1.27 1.27)) (justify left))
     )
-    (property "Footprint" "Connector_PinHeader_2.54mm:PinHeader_1x01_P2.54mm_Vertical" (id 2) (at 93.98 39.37 0)
-      (effects (font (size 1.27 1.27)) hide)
-    )
+    (property "Footprint" "TestPoint:TestPoint_Pad_2.5x2.5mm" (id 2) (at 93.98 39.37 0)
+      (effects (font (size 1.27 1.27)) hide)
+    )
