File: baremetal/WindowViewer_Battery/kicad/ESP32_BAT/sensor.kicad_sch (KiCad schematic)
At the start: 0 parts

Commit message: battery pcb update, schematic done
Parts:
- added C10: 22pf, Capacitor_SMD:C_1206_3216Metric_Pad1.33x1.80mm_HandSolder, symbol Device:C
- added C11, C9: 200nf, Capacitor_SMD:C_1206_3216Metric_Pad1.33x1.80mm_HandSolder, symbol Device:C
- added J3: Conn_01x03_Male, Connector_PinHeader_2.54mm:PinHeader_1x03_P2.54mm_Vertical, symbol Connector:Conn_01x03_Male
- added Q1: BC817, Package_TO_SOT_SMD:SOT-23, symbol Transistor_BJT:BC817
- added R11: 4.7k, Resistor_SMD:R_1206_3216Metric_Pad1.30x1.75mm_HandSolder, symbol Device:R
- added R12, R13, R15: 0, Resistor_SMD:R_1206_3216Metric_Pad1.30x1.75mm_HandSolder, symbol Device:R
- added R14: 100k, Resistor_SMD:R_1206_3216Metric_Pad1.30x1.75mm_HandSolder, symbol Device:R
- added U3: am2320, Connector_PinHeader_2.54mm:PinHeader_1x04_P2.54mm_Vertical, symbol gliese:am2320
Connections:
- new net: Q1.1 (B), R11.1
- new net: J3.2 (Pin_2), R14.2
- new net +3V3: C10.1, C9.1, J3.3 (Pin_3), U3.1 (VDD)
- new net ADC_SNS_IN: C11.1, R14.1
- new net CLK: U3.4 (SCL)
- new net GND: Q1.2 (E), R12.2, R13.2, R15.2
- new net SDA: U3.2 (SDA)
- new net SENSOR_ON: R11.2
- new net sensor_gnd: C10.2, C11.2, C9.2, J3.1 (Pin_1), Q1.3 (C), R12.1, R13.1, R15.1, U3.3 (GND)

Commit message: watersensor 0.1
Parts:
- removed R13: 0, Resistor_SMD:R_1206_3216Metric_Pad1.30x1.75mm_HandSolder, symbol Device:R
Changed lines of the file:
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@@
   (junction (at 203.2 52.07) (diameter 0) (color 0 0 0 0)
-  )
-  (junction (at 203.2 73.66) (diameter 0) (color 0 0 0 0)
   )
   (junction (at 224.79 54.61) (diameter 0) (color 0 0 0 0)
@@
     (pin "2")
   )
-  (symbol (lib_id "power:GND") (at 203.2 81.28 0) (unit 1)
-    (in_bom yes) (on_board yes) (fields_autoplaced)
-    (property "Reference" "#PWR0135" (id 0) (at 203.2 87.63 0)
-      (effects (font (size 1.27 1.27)) hide)
-    )
-    (property "Value" "GND" (id 1) (at 203.2 86.36 0))
-    (property "Footprint" "" (id 2) (at 203.2 81.28 0)
-      (effects (font (size 1.27 1.27)) hide)
-    )
-    (property "Datasheet" "" (id 3) (at 203.2 81.28 0)
-      (effects (font (size 1.27 1.27)) hide)
-    )
-    (pin "1")
-  )
   (symbol (lib_id "Device:R") (at 49.53 93.98 270) (unit 1)
     (in_bom yes) (on_board yes)
@@
     (pin "3")
   )
-  (symbol (lib_id "Device:R") (at 203.2 77.47 0) (unit 1)
-    (in_bom yes) (on_board yes)
-    (property "Reference" "R13" (id 0) (at 197.9422 77.47 90))
-    (property "Value" "0" (id 1) (at 200.2536 77.47 90))
-    (property "Footprint" "Resistor_SMD:R_1206_3216Metric_Pad1.30x1.75mm_HandSolder" (id 2) (at 201.422 77.47 90)
-      (effects (font (size 1.27 1.27)) hide)
-    )
-    (property "Datasheet" "~" (id 3) (at 203.2 77.47 0)
-      (effects (font (size 1.27 1.27)) hide)
-    )
-    (pin "1")
-    (pin "2")
-  )
   (symbol (lib_id "power:GND") (at 128.27 81.28 0) (unit 1)
